File: macro4x4.sch (KiCad schematic (older format))
At the start: 34 parts, among them SW1 SW_Push, SW10 SW_Push, SW11 SW_Push, SW12 SW_Push, SW13 SW_Push, SW14 SW_Push, SW15 SW_Push, SW16 SW_Push, SW2 SW_Push, SW3 SW_Push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

Commit message: ・回路図を修正 ・基板でビアを使用しないように修正
Changed lines of the file:
@@
 Text GLabel 3600 3900 0    50   Input ~ 0
 ROW3
-Text GLabel 4050 1100 1    50   Input ~ 0
+Text GLabel 4050 1100 1    50   Output ~ 0
 COL0
-Text GLabel 4850 1100 1    50   Input ~ 0
+Text GLabel 4850 1100 1    50   Output ~ 0
 COL1
-Text GLabel 5600 1100 1    50   Input ~ 0
+Text GLabel 5600 1100 1    50   Output ~ 0
 COL2
-Text GLabel 6300 1100 1    50   Input ~ 0
+Text GLabel 6300 1100 1    50   Output ~ 0
 COL3
-Text GLabel 2250 1950 2    50   Input ~ 0
+Text GLabel 2250 1950 2    50   Output ~ 0
 ROW0
-Text GLabel 2250 2050 2    50   Input ~ 0
+Text GLabel 2250 2050 2    50   Output ~ 0
 ROW1
-Text GLabel 2250 2150 2    50   Input ~ 0
+Text GLabel 2250 2150 2    50   Output ~ 0
 ROW2
-Text GLabel 2250 2250 2    50   Input ~ 0
+Text GLabel 2250 2250 2    50   Output ~ 0
 ROW3
 Text GLabel 2250 2450 2    50   Input ~ 0
